File: eagle/slider.brd (EAGLE design)
At the start: 68.2 x 43.2 mm, 9 parts

Commit message: Schematic fixups
Parts:
- added J2: (no value), ELFIN:GMKDS1,5
Connections:
- new net ENDSTOP: J2.1, U$1.JP2.4
- net GND: now also J2.2
Routing:
- net ENDSTOP: track 0.00 -> 8.25 mm
Other:
- board size 68.2 x 43.2 mm -> 73.3 x 43.2 mm
Changed lines of the file:
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@@
 <board>
 <plain>
-<wire x1="0" y1="0" x2="68.25" y2="0" width="0" layer="20"/>
-<wire x1="68.25" y1="0" x2="68.25" y2="43.17" width="0" layer="20"/>
-<wire x1="68.25" y1="43.17" x2="0" y2="43.17" width="0" layer="20"/>
+<wire x1="0" y1="0" x2="73.33" y2="0" width="0" layer="20"/>
+<wire x1="73.33" y1="0" x2="73.33" y2="43.17" width="0" layer="20"/>
+<wire x1="73.33" y1="43.17" x2="0" y2="43.17" width="0" layer="20"/>
 <wire x1="0" y1="43.17" x2="0" y2="0" width="0" layer="20"/>
 </plain>
@@
 <element name="R2" library="SMD" package="0805" value="1k" x="64.77" y="26.67" rot="MR90"/>
 <element name="C1" library="DISCRETE_mm" package="ES-3,5/8" value="100u/16V" x="13.97" y="35.56" rot="R180"/>
+<element name="J2" library="ELFIN" package="GMKDS1,5" value="" x="68.58" y="15.24"/>
 </elements>
 <signals>
@@
 <polygon width="1.016" layer="16" isolate="0.8128">
 <vertex x="1.27" y="41.91"/>
-<vertex x="67.31" y="41.91"/>
-<vertex x="67.31" y="1.27"/>
+<vertex x="72.39" y="41.91"/>
+<vertex x="72.39" y="1.27"/>
 <vertex x="1.27" y="1.27"/>
 </polygon>
 <contactref element="C1" pad="2"/>
-<wire x1="21.59" y1="30.48" x2="26.43" y2="40.64" width="0" layer="19" extent="16-16"/>
+<contactref element="J2" pad="2"/>
 </signal>
 <signal name="+3.3V">
@@
 <wire x1="60.96" y1="25.4" x2="60.96" y2="24.765" width="1.016" layer="16"/>
 </signal>
+<signal name="ENDSTOP">
+<contactref element="U$1" pad="JP2.4"/>
+<contactref element="J2" pad="1"/>
+<wire x1="60.96" y1="19.685" x2="68.58" y2="19.685" width="1.016" layer="16"/>
+<wire x1="68.58" y1="19.685" x2="68.58" y2="19.05" width="1.016" layer="16"/>
+</signal>
 </signals>
