File: eagle/slider.sch (EAGLE design)
At the start: 9 parts

Commit message: Schematic fixups
Parts:
- added J2: (no value), ELFIN:GMKDS-2
Connections:
- new net ENDSTOP: J2.1, U$1.D2
- net GND: now also J2.2
Changed lines of the file:
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@@
 <part name="C1" library="DISCRETE_mm" deviceset="C-EL" device="-3,5/8" value="100u/16V"/>
 <part name="U$4" library="SUPPLY" deviceset="GND" device=""/>
+<part name="J2" library="ELFIN" deviceset="GMKDS-2" device=""/>
+<part name="U$7" library="SUPPLY" deviceset="GND" device=""/>
 </parts>
 <sheets>
@@
 <instance part="C1" gate="C" x="27.94" y="2.54"/>
 <instance part="U$4" gate="GND" x="27.94" y="-5.08"/>
+<instance part="J2" gate="G$1" x="121.92" y="58.42"/>
+<instance part="U$7" gate="GND" x="114.3" y="53.34"/>
 </instances>
 <busses>
@@
 <pinref part="C1" gate="C" pin="2"/>
 <pinref part="U$4" gate="GND" pin="GND"/>
+</segment>
+<segment>
+<pinref part="J2" gate="G$1" pin="2"/>
+<pinref part="U$7" gate="GND" pin="GND"/>
 </segment>
 </net>
@@
 </segment>
 </net>
+<net name="ENDSTOP" class="0">
+<segment>
+<pinref part="U$1" gate="G$1" pin="D2"/>
+<wire x1="86.36" y1="58.42" x2="111.76" y2="58.42" width="0.1524" layer="91"/>
+<wire x1="111.76" y1="58.42" x2="111.76" y2="60.96" width="0.1524" layer="91"/>
+<pinref part="J2" gate="G$1" pin="1"/>
+<wire x1="111.76" y1="60.96" x2="114.3" y2="60.96" width="0.1524" layer="91"/>
+<label x="91.44" y="58.42" size="1.778" layer="95"/>
+</segment>
+</net>
